File: teclado_matricial2/teclado_matricial.kicad_pcb (KiCad board)
At the start: 2 copper layers, 138.2 x 57 mm, 31 parts

Commit message: New Day
Other:
- board size 138.2 x 57 mm -> 138 x 57 mm
Changed lines of the file:
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@@
 	(gr_line
 		(start 217.5 133)
-		(end 79.25 133)
+		(end 79.5 133)
 		(stroke
 			(width 0.05)
