File: pcb geral/pcb_geral.kicad_pcb (KiCad board)
At the start: 2 copper layers, 138.2 x 57 mm, 4 parts

Commit message: New Day
Parts:
- removed the REF** at (138.5, 96.0)
- added REF**: MountingHole_2.5mm, MountingHole:MountingHole_2.5mm, F.Cu at (90.8, 99.2)
Connections:
- REF** pad 1: (no net) -> .
- REF** pad 10: (no net) -> .
Routing:
- net (no net): track 646.0 -> 1034.1 mm
- net .: track 1508.7 -> 1560.2 mm, vias 10 -> 6
Other:
- board size 138.2 x 57 mm -> 138 x 57 mm
- board text added: "45"
- board text removed: "49"

Commit message: Another Day of Work
Parts:
- added REF**: TE_1-84952-4_1x14-1MP_P1.0mm_Horizontal, Connector_FFC-FPC:TE_1-84952-4_1x14-1MP_P1.0mm_Horizontal, F.Cu at (98.0, 84.0)
- added REF**: PinHeader_1x14_P1.00mm_Vertical, Connector_PinHeader_1.00mm:PinHeader_1x14_P1.00mm_Vertical, F.Cu at (91.2, 89.1)
- moved REF** 3.44 mm to (90.8, 102.7)
Routing:
- net (no net): track 1034.1 -> 1071.9 mm, vias 26 -> 22
- net .: track 1560.2 -> 1555.2 mm
Other:
- board text added: "4 sd"
