File: unified pcb/kicad/razor32.kicad_pcb (KiCad board)
At the start: 4 copper layers, 138 x 57 mm, 33 parts

Commit message: pcb
Connections:
- ESP32PinSocket_1 pad 11: (no net) -> .
- ESP32PinSocket_1 pad 12: (no net) -> .
- ESP32PinSocket_1 pad 13: (no net) -> .
- ESP32PinSocket_2 pad 10: . -> (no net)
- ESP32PinSocket_2 pad 11: . -> (no net)
- ESP32PinSocket_2 pad 9: . -> (no net)
Routing:
- net .: track 2032.3 -> 2172.0 mm

Commit message: pcb nets
Connections:
- ESP32PinSocket_1 pad 10: . -> y1
- ESP32PinSocket_1 pad 11: . -> x6
- ESP32PinSocket_1 pad 12: . -> x3
- ESP32PinSocket_1 pad 13: . -> x4
- ESP32PinSocket_1 pad 6: . -> x10
- ESP32PinSocket_2 pad 13: . -> x8
- ESP32PinSocket_2 pad 14: . -> x5
- ESP32PinSocket_2 pad 15: . -> y3
- ESP32PinSocket_2 pad 16: . -> x7
- ESP32PinSocket_2 pad 4: . -> y2
- ESP32PinSocket_2 pad 5: . -> x9
- ESP32PinSocket_2 pad 6: . -> x1
- ESP32PinSocket_2 pad 7: . -> x2
- a pad 2: . -> x1
- b pad 2: . -> x5
- c pad 2: . -> x3
- d pad 2: . -> x3
- e pad 2: . -> x3
- enter pad 2: . -> x10
- f pad 2: . -> x4
- fun pad 2: . -> x9
- g pad 2: . -> x5
- h pad 2: . -> x6
- i pad 2: . -> x8
- j pad 2: . -> x7
- k pad 2: . -> x8
- l pad 2: . -> x9
- m pad 2: . -> x8
- n pad 2: . -> x7
- o pad 2: . -> x9
- p pad 2: . -> x10
- q pad 2: . -> x1
- r pad 2: . -> x4
- ret pad 2: . -> x10
- s pad 2: . -> x2
- space pad 2: . -> x6
- t pad 2: . -> x5
- u pad 2: . -> x7
- v pad 2: . -> x4
- w pad 2: . -> x2
- x pad 2: . -> x2
- y pad 2: . -> x6
- z pad 2: . -> x1
Routing:
- net .: track 2172.0 -> 0.00 mm, vias 6 -> 0
- net x6: track 0.00 -> 292.0 mm, vias 0 -> 1
- net x4: track 0.00 -> 281.1 mm, vias 0 -> 1
- net x3: track 0.00 -> 265.5 mm, vias 0 -> 1
- net x5: track 0.00 -> 254.4 mm, vias 0 -> 1
- net x2: track 0.00 -> 214.9 mm, vias 0 -> 1
- net x1: track 0.00 -> 207.2 mm, vias 0 -> 1
- net y1: track 0.00 -> 201.4 mm
- net y3: track 0.00 -> 160.9 mm
- net y2: track 0.00 -> 140.1 mm
- net x10: track 0.00 -> 57.3 mm
- net x8: track 0.00 -> 38.2 mm
- net x9: track 0.00 -> 30.3 mm
- net x7: track 0.00 -> 29.0 mm
