File: unified pcb/kicad/razor32.kicad_pcb (KiCad board)
At the start: 4 copper layers, 138 x 57 mm, 33 parts

Commit message: asf
Connections:
- ESP32PinSocket_1 pad 15: (no net) -> x10
- ESP32PinSocket_1 pad 6: x10 -> (no net)
Routing:
- net x10: track 57.3 -> 79.9 mm, vias 0 -> 1
- net y3: track 160.9 -> 160.2 mm

Commit message: add
Connections:
- a pad 1: gnd -> y2
- b pad 1: gnd -> y3
- c pad 1: gnd -> y3
- d pad 1: gnd -> y2
- e pad 1: gnd -> y1
- enter pad 1: gnd -> y3
- f pad 1: gnd -> y2
- fun pad 1: gnd -> y3
- g pad 1: gnd -> y2
- h pad 1: gnd -> y2
- i pad 1: gnd -> y1
- j pad 1: gnd -> y2
- k pad 1: gnd -> y2
- l pad 1: gnd -> y2
- m pad 1: gnd -> y3
- n pad 1: gnd -> y3
- o pad 1: gnd -> y1
- p pad 1: gnd -> y1
- q pad 1: gnd -> y1
- r pad 1: gnd -> y1
- ret pad 1: gnd -> y2
- s pad 1: gnd -> y2
- space pad 1: gnd -> y3
- t pad 1: gnd -> y1
- u pad 1: gnd -> y1
- v pad 1: gnd -> y3
- w pad 1: gnd -> y1
- x pad 1: gnd -> y3
- y pad 1: gnd -> y1
- z pad 1: gnd -> y3
Routing:
- net gnd: track 543.7 -> 0.00 mm
- net y1: track 201.4 -> 227.2 mm, vias 0 -> 20
- net y2: track 140.1 -> 162.7 mm, vias 0 -> 20
- net x8: track 38.2 -> 58.7 mm, vias 0 -> 6
- net y3: track 160.2 -> 180.1 mm, vias 0 -> 21
- net x6: track 292.0 -> 311.7 mm, vias 1 -> 7
- net x9: track 30.3 -> 47.4 mm, vias 0 -> 6
- net x10: track 79.9 -> 96.5 mm, vias 1 -> 7
- net x1: track 207.2 -> 223.7 mm, vias 1 -> 7
- net x7: track 29.0 -> 44.4 mm, vias 0 -> 6
- net x2: track 214.9 -> 230.0 mm, vias 1 -> 7
- net x4: track 281.1 -> 296.1 mm, vias 1 -> 7
- net x5: track 254.4 -> 269.3 mm, vias 1 -> 7
- net x3: track 265.5 -> 279.5 mm, vias 1 -> 7
- net bl: track 186.4 -> 184.7 mm
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Other:
- board text added: "^"
