File: unified pcb/kicad/razor32.kicad_sch (KiCad schematic)
At the start: 66 parts, among them J1 ESP32 Connector_1, J2 ESP32 Connector_2, J3 Keyboard Connector_1, J4 Keyboard Connector_2, J5 Flat Cable Header, J6 FLAT CABLE SOCKET, SW1 PushButton 6mm 4pin, SW10 PushButton 6mm 4pin, SW11 PushButton 6mm 4pin, SW12 PushButton 6mm 4pin, SW13 PushButton 6mm 4pin, SW14 PushButton 6mm 4pin, SW15 PushButton 6mm 4pin, SW16 PushButton 6mm 4pin, SW17 PushButton 6mm 4pin, SW18 PushButton 6mm 4pin, SW19 PushButton 6mm 4pin, SW2 PushButton 6mm 4pin, SW20 PushButton 6mm 4pin, SW21 PushButton 6mm 4pin, SW22 PushButton 6mm 4pin, SW23 PushButton 6mm 4pin, SW24 PushButton 6mm 4pin, SW25 PushButton 6mm 4pin, SW26 PushButton 6mm 4pin, SW27 PushButton 6mm 4pin, SW28 PushButton 6mm 4pin, SW29 PushButton 6mm 4pin, SW3 PushButton 6mm 4pin, SW30 PushButton 6mm 4pin, SW31 PushButton 6mm 4pin, SW32 PushButton 6mm 4pin, SW33 PushButton 6mm 4pin, SW34 PushButton 6mm 4pin, SW35 PushButton 6mm 4pin, SW36 PushButton 6mm 4pin, SW37 PushButton 6mm 4pin, SW38 PushButton 6mm 4pin, SW39 PushButton 6mm 4pin, SW4 PushButton 6mm 4pin, SW40 PushButton 6mm 4pin, SW41 PushButton 6mm 4pin, SW42 PushButton 6mm 4pin, SW43 PushButton 6mm 4pin, SW44 PushButton 6mm 4pin, SW45 PushButton 6mm 4pin, SW46 PushButton 6mm 4pin, SW47 PushButton 6mm 4pin, SW48 PushButton 6mm 4pin, SW49 PushButton 6mm 4pin, SW5 PushButton 6mm 4pin, SW50 PushButton 6mm 4pin, SW51 PushButton 6mm 4pin, SW52 PushButton 6mm 4pin, SW53 PushButton 6mm 4pin, SW54 PushButton 6mm 4pin, SW55 PushButton 6mm 4pin, SW56 PushButton 6mm 4pin, SW57 PushButton 6mm 4pin, SW58 PushButton 6mm 4pin, SW59 PushButton 6mm 4pin, SW6 PushButton 6mm 4pin, SW60 PushButton 6mm 4pin, SW7 PushButton 6mm 4pin, SW8 PushButton 6mm 4pin, SW9 PushButton 6mm 4pin

Commit message: add
Parts:
- added D1, D10, D11, D12, D13, D14, D15, D16, D17, D18, D19, D2, D20, D21, D22, D23, D24, D25, D26, D27, D28, D29, D3, D30, D31, D32, D33, D34, D35, D36, D37, D38, D39, D4, D40, D41, D42, D43, D44, D45, D46, D47, D48, D49, D5, D50, D51, D52, D53, D54, D55, D56, D57, D58, D59, D6, D60, D7, D8, D9: 1N4007, Diode_THT:D_DO-41_SOD81_P10.16mm_Horizontal, symbol Diode:1N4007
Connections:
- net GND: no longer SW1.1, SW10.1, SW11.1, SW12.1, SW13.1, SW14.1, SW15.1, SW16.1, SW17.1, SW18.1, SW19.1, SW2.1, SW20.1, SW21.1, SW22.1, SW23.1, SW24.1, SW25.1, SW26.1, SW27.1, SW28.1, SW29.1, SW3.1, SW30.1, SW31.1, SW32.1, SW33.1, SW34.1, SW35.1, SW36.1, SW37.1, SW38.1, SW39.1, SW4.1, SW40.1, SW41.1, SW42.1, SW43.1, SW44.1, SW45.1, SW46.1, SW47.1, SW48.1, SW5.1, SW50.1, SW51.1, SW52.1, SW53.1, SW54.1, SW55.1, SW56.1, SW57.1, SW58.1, SW59.1, SW6.1, SW60.1, SW7.1, SW8.1, SW9.1
- net X1: now also D1.1 (K), D2.1 (K), D3.1 (K); no longer SW1.4, SW2.4, SW3.4
- net X10: now also D28.1 (K), D29.1 (K), D30.1 (K); no longer SW28.4, SW29.4, SW30.4
- net X2: now also D4.1 (K), D5.1 (K), D6.1 (K); no longer SW4.4, SW5.4, SW6.4
- net X3: now also D7.1 (K), D8.1 (K), D9.1 (K); no longer SW7.4, SW8.4, SW9.4
- net X4: now also D10.1 (K), D11.1 (K), D12.1 (K); no longer SW10.4, SW11.4, SW12.4
- net X5: now also D13.1 (K), D14.1 (K), D15.1 (K); no longer SW13.4, SW14.4, SW15.4
- net X6: now also D16.1 (K), D17.1 (K), D18.1 (K); no longer SW16.4, SW17.4, SW18.4
- net X7: now also D19.1 (K), D20.1 (K), D21.1 (K); no longer SW19.4, SW20.4, SW21.4
- net X8: now also D22.1 (K), D23.1 (K), D24.1 (K); no longer SW22.4, SW23.4, SW24.4
- net X9: now also D25.1 (K), D26.1 (K), D27.1 (K); no longer SW25.4, SW26.4, SW27.4
- net Y1: now also D31.2 (A), D32.2 (A), D33.2 (A), D34.2 (A), D35.2 (A), D36.2 (A), D37.2 (A), D38.2 (A), D39.2 (A), D60.2 (A); no longer SW31.4, SW34.4, SW37.4, SW40.4, SW43.4, SW46.4, SW49.4, SW52.4, SW55.4, SW58.4
- net Y2: now also D40.2 (A), D41.2 (A), D42.2 (A), D43.2 (A), D44.2 (A), D45.2 (A), D46.2 (A), D47.2 (A), D48.2 (A), D49.2 (A); no longer SW32.4, SW35.4, SW38.4, SW41.4, SW44.4, SW47.4, SW50.4, SW53.4, SW56.4, SW59.4
- net Y3: now also D50.2 (A), D51.2 (A), D52.2 (A), D53.2 (A), D54.2 (A), D55.2 (A), D56.2 (A), D57.2 (A), D58.2 (A), D59.2 (A); no longer SW33.4, SW36.4, SW39.4, SW42.4, SW45.4, SW48.4, SW51.4, SW54.4, SW57.4, SW60.4
- new net: D47.1 (K), SW53.4
- new net: D1.2 (A), SW2.1
- new net: D11.2 (A), SW11.1
- new net: D21.2 (A), SW21.1
- new net: D46.1 (K), SW50.4
- new net: D8.2 (A), SW8.1
- new net: D34.1 (K), SW40.4
- new net: D5.2 (A), SW5.1
- new net: D24.2 (A), SW24.1
- new net: D59.1 (K), SW60.4
- new net: D29.2 (A), SW29.1
- new net: D38.1 (K), SW55.4
- new net: D4.2 (A), SW4.1
- new net: D9.2 (A), SW9.1
- new net: D43.1 (K), SW41.4
- new net: D30.2 (A), SW30.1
- new net: D58.1 (K), SW57.4
- new net: D44.1 (K), SW44.4
- new net: D25.2 (A), SW25.1
- new net: D60.1 (K), SW43.4
- new net: D54.1 (K), SW45.4
- new net: D7.2 (A), SW7.1
- new net: D23.2 (A), SW23.1
- new net: D19.2 (A), SW19.1
- new net: D35.1 (K), SW46.4
- new net: D2.2 (A), SW1.1
- new net: D20.2 (A), SW20.1
- new net: D16.2 (A), SW16.1
- new net: D6.2 (A), SW6.1
- new net: D32.1 (K), SW34.4
- new net: D49.1 (K), SW59.4
- new net: D39.1 (K), SW58.4
- new net: D57.1 (K), SW54.4
- new net: D31.1 (K), SW31.4
- new net: D40.1 (K), SW32.4
- new net: D53.1 (K), SW42.4
- new net: D14.2 (A), SW14.1
- new net: D51.1 (K), SW36.4
- new net: D13.2 (A), SW13.1
- new net: D42.1 (K), SW38.4
- new net: D41.1 (K), SW35.4
- new net: D15.2 (A), SW15.1
- new net: D26.2 (A), SW26.1
- new net: D28.2 (A), SW28.1
- new net: D56.1 (K), SW51.4
- new net: D50.1 (K), SW33.4
- new net: D12.2 (A), SW12.1
- new net: D36.1 (K), SW49.4
- new net: D37.1 (K), SW52.4
- new net: D48.1 (K), SW56.4
- new net: D22.2 (A), SW22.1
- new net: D3.2 (A), SW3.1
- new net: D45.1 (K), SW47.4
- new net: D33.1 (K), SW37.4
- new net: D27.2 (A), SW27.1
- new net: D55.1 (K), SW48.4
- new net: D18.2 (A), SW18.1
- new net: D17.2 (A), SW17.1
- new net: D10.2 (A), SW10.1
- new net: D52.1 (K), SW39.4
Other:
- note added: "Y pin: INPUT_PULLUP X pin: INPUT"
- note removed: "Buttons work as push up. GND is given to the push button left upper pin and when it is pressed, ground flows through the right lower pin, triggering push up in ESP32 GPIO."
- note removed: "Keyboard will be connected using pin headers and sockets"

Commit message: pcb
Parts:
- removed D58, D59: 1N4007, Diode_THT:D_DO-41_SOD81_P10.16mm_Horizontal, symbol Diode:1N4007
- added D61, D62: 1N4007, Diode_THT:D_DO-41_SOD81_P10.16mm_Horizontal, symbol Diode:1N4007
Connections:
- net X2: no longer D6.1 (K)
- net Y2: now also D61.2 (A); no longer D49.2 (A)
- net Y3: now also D49.2 (A), D62.2 (A)
- net at SW53.1: now also D47.1 (K)
- net at SW53.4: no longer D47.1 (K)
- net at D1.2 (A): now also SW2.4; no longer SW2.1
- net at D11.2 (A): now also SW11.4; no longer SW11.1
- net at SW21.1: no longer D21.2 (A)
- net at SW21.4: now also D21.2 (A)
- net at D46.1 (K): now also SW50.1; no longer SW50.4
- net at SW8.1: no longer D8.2 (A)
- net at SW8.4: now also D8.2 (A)
- net at D34.1 (K): now also SW40.1; no longer SW40.4
- net at SW5.1: no longer D5.2 (A)
- net at SW5.4: now also D5.2 (A)
- net at SW24.1: no longer D24.2 (A)
- net at SW24.4: now also D24.2 (A)
- net at SW29.1: no longer D29.2 (A)
- net at SW29.4: now also D29.2 (A)
- net at SW55.4: no longer D38.1 (K)
- net at D4.2 (A): now also SW4.4; no longer SW4.1
- net at SW9.1: no longer D9.2 (A)
- net at SW9.4: now also D9.2 (A)
- net at SW41.1: now also D43.1 (K)
- net at SW41.4: no longer D43.1 (K)
- net at SW30.1: no longer D30.2 (A)
- net at SW57.1: now also D57.1 (K)
- net at SW60.1: now also D62.1 (K)
- net at SW44.1: now also D44.1 (K)
- net at SW44.4: no longer D44.1 (K)
- net at SW25.1: no longer D25.2 (A)
- net at SW55.1: now also D39.1 (K)
- net at SW43.1: now also D35.1 (K)
- net at SW43.4: no longer D60.1 (K)
- net at SW45.1: now also D53.1 (K)
- net at SW45.4: no longer D54.1 (K)
- net at D7.2 (A): now also SW7.4; no longer SW7.1
- net at D23.2 (A): now also SW23.4; no longer SW23.1
- net at D19.2 (A): now also SW19.4; no longer SW19.1
- net at SW46.1: now also D36.1 (K)
- net at SW46.4: no longer D35.1 (K)
- net at SW1.1: no longer D2.2 (A)
- net at SW1.4: now also D2.2 (A)
- net at D20.2 (A): now also SW20.4; no longer SW20.1
- net at SW16.1: no longer D16.2 (A)
- net at D6.2 (A): now also SW6.4; no longer SW6.1
- net at D32.1 (K): now also SW34.1; no longer SW34.4
- net at SW59.1: now also D61.1 (K)
- net at SW59.4: no longer D49.1 (K)
- net at SW58.4: no longer D39.1 (K)
- net at SW54.1: now also D56.1 (K)
- net at SW54.4: no longer D57.1 (K)
- net at D31.1 (K): now also SW31.1; no longer SW31.4
- net at SW32.1: now also D40.1 (K)
- net at SW32.4: no longer D40.1 (K)
- net at SW42.1: now also D52.1 (K)
- net at SW42.4: no longer D53.1 (K)
- net at SW14.1: no longer D14.2 (A)
- net at SW14.4: now also D14.2 (A)
- net at SW58.1: now also D60.1 (K)
- net at SW36.1: now also D50.1 (K)
- net at D51.1 (K): now also SW39.1; no longer SW36.4
- net at D13.2 (A): now also SW13.4; no longer SW13.1
- net at D42.1 (K): now also SW38.1; no longer SW38.4
- net at SW35.1: now also D41.1 (K)
- net at SW35.4: no longer D41.1 (K)
- net at SW15.1: no longer D15.2 (A)
- net at D26.2 (A): now also SW26.4; no longer SW26.1
- net at D28.2 (A): now also SW28.4; no longer SW28.1
- net at SW51.1: now also D55.1 (K)
- net at SW51.4: no longer D56.1 (K)
- net at SW33.1: now also D49.1 (K)
- net at SW33.4: no longer D50.1 (K)
- net at D12.2 (A): now also SW12.4; no longer SW12.1
- net at SW49.1: now also D37.1 (K)
- net at SW49.4: no longer D36.1 (K)
- net at SW52.4: no longer D37.1 (K)
- net at SW56.1: now also D48.1 (K)
- net at SW56.4: no longer D48.1 (K)
- net at D22.2 (A): now also SW22.4; no longer SW22.1
- net at SW3.1: no longer D3.2 (A)
- net at D45.1 (K): now also SW47.1; no longer SW47.4
- net at SW3.4: now also D3.2 (A)
- net at SW37.1: now also D33.1 (K)
- net at SW37.4: no longer D33.1 (K)
- net at D27.2 (A): now also SW27.4; no longer SW27.1
- net at SW15.4: now also D15.2 (A)
- net at SW48.1: now also D54.1 (K)
- net at SW48.4: no longer D55.1 (K)
- net at SW18.1: no longer D18.2 (A)
- net at SW18.4: now also D18.2 (A)
- net at SW25.4: now also D25.2 (A)
- net at SW17.1: no longer D17.2 (A)
- net at SW17.4: now also D17.2 (A)
- net at SW10.1: no longer D10.2 (A)
- net at SW10.4: now also D10.2 (A)
- net at SW52.1: now also D38.1 (K)
- net at SW16.4: now also D16.2 (A)
- net at SW39.4: no longer D52.1 (K)
- net at SW30.4: now also D30.2 (A)
