File: unified pcb/kicad/razor32.kicad_sch (KiCad schematic)
At the start: 96 parts, among them J1 ESP32 Connector_1, J2 ESP32 Connector_2, J3 Keyboard Connector_1, J4 Keyboard Connector_2, J5 Flat Cable Header, J6 FLAT CABLE SOCKET, SW1 PushButton 6mm 4pin, SW10 PushButton 6mm 4pin, SW11 PushButton 6mm 4pin, SW12 PushButton 6mm 4pin, SW13 PushButton 6mm 4pin, SW14 PushButton 6mm 4pin, SW15 PushButton 6mm 4pin, SW16 PushButton 6mm 4pin, SW17 PushButton 6mm 4pin, SW18 PushButton 6mm 4pin, SW19 PushButton 6mm 4pin, SW2 PushButton 6mm 4pin, SW20 PushButton 6mm 4pin, SW21 PushButton 6mm 4pin, SW22 PushButton 6mm 4pin, SW23 PushButton 6mm 4pin, SW24 PushButton 6mm 4pin, SW25 PushButton 6mm 4pin, SW26 PushButton 6mm 4pin, SW27 PushButton 6mm 4pin, SW28 PushButton 6mm 4pin, SW29 PushButton 6mm 4pin, SW3 PushButton 6mm 4pin, SW30 PushButton 6mm 4pin, SW4 PushButton 6mm 4pin, SW5 PushButton 6mm 4pin, SW6 PushButton 6mm 4pin, SW7 PushButton 6mm 4pin, SW8 PushButton 6mm 4pin, SW9 PushButton 6mm 4pin

Commit message: Clean PCB
Parts:
- removed D1, D10, D11, D12, D13, D14, D15, D16, D17, D18, D19, D2, D20, D21, D22, D23, D24, D25, D26, D27, D28, D29, D3, D30, D4, D5, D6, D7, D8, D9: 1N4007, Diode_THT:D_DO-41_SOD81_P10.16mm_Horizontal, symbol Diode:1N4007
Connections:
- net X1: now also SW1.4, SW2.4, SW3.4
- net X10: now also SW28.4, SW29.4, SW30.4
- net X2: now also SW4.4, SW5.4, SW6.4
- net X3: now also SW7.4, SW8.4, SW9.4
- net X4: now also SW10.4, SW11.4, SW12.4
- net X5: now also SW13.4, SW14.4, SW15.4
- net X6: now also SW16.4, SW17.4, SW18.4
- net X7: now also SW19.4, SW20.4, SW21.4
- net X8: now also SW22.4, SW23.4, SW24.4
- net X9: now also SW25.4, SW26.4, SW27.4
Other:
- note added: "Y pin: INPUT_PULLUP X pin: INPUT/OUTPUT"
- note removed: "Y pin: INPUT_PULLUP X pin: INPUT"
